Commit message: Alternative Approach - v1

File: urdf/onrobot_2fg7.trans.xacro (robot description, xacro)
@@ -1,15 +1,15 @@
 <?xml version="1.0" encoding="UTF-8"?>
-<robot xmlns:xacro="http://ros.org/wiki/xacro" name = 'transmission'>
+<robot xmlns:xacro="http://ros.org/wiki/xacro" name='transmission'>
   <xacro:macro name="gripper_transmission">
-      <transmission name="left_finger_joint_tran">
-        <type>transmission_interface/SimpleTransmission</type>
-          <joint name="left_finger_joint">
-            <hardwareInterface>hardware_interface/PositionJointInterface</hardwareInterface>
-          </joint>
-        <actuator name="left_finger_joint_motor">
-          <hardwareInterface>hardware_interface/PositionJointInterface</hardwareInterface>
-          <mechanicalReduction>1</mechanicalReduction>
-        </actuator>
-      </transmission>
+    <transmission name="left_finger_joint_tran">
+      <type>transmission_interface/SimpleTransmission</type>
+      <joint name="left_finger_joint">
+        <hardwareInterface>hardware_interface/PositionJointInterface</hardwareInterface>
+      </joint>
+      <actuator name="left_finger_joint_motor">
+        <hardwareInterface>hardware_interface/PositionJointInterface</hardwareInterface>
+        <mechanicalReduction>1</mechanicalReduction>
+      </actuator>
+    </transmission>
   </xacro:macro>
 </robot>

Commit message: URDF Transmission Issues

File: urdf/onrobot_2fg7.trans.xacro (robot description, xacro)
@@ -12,4 +12,14 @@
       </actuator>
     </transmission>
+    <transmission name="right_finger_joint_tran">
+      <type>transmission_interface/SimpleTransmission</type>
+      <joint name="right_finger_joint">
+        <hardwareInterface>hardware_interface/PositionJointInterface</hardwareInterface>
+      </joint>
+      <actuator name="right_finger_joint_motor">
+        <hardwareInterface>hardware_interface/PositionJointInterface</hardwareInterface>
+        <mechanicalReduction>1</mechanicalReduction>
+      </actuator>
+    </transmission>
   </xacro:macro>
 </robot>
