Commit message: ROS2 Migration - Fix

File: urdf/onrobot_2fg7.xacro (robot description, xacro)
@@ -18,5 +18,5 @@
         <origin xyz="0 0 0" rpy="0 0 0"/>
         <geometry>
-          <mesh filename="package://onrobot_2fg7_description/meshes/base_link.stl" scale="0.001 0.001 0.001"/>
+          <mesh filename="package://onrobot_2fg7_description/urdf/meshes/base_link.stl" scale="0.001 0.001 0.001"/>
         </geometry>
         <material name="silver"/>
@@ -25,5 +25,5 @@
         <origin xyz="0 0 0" rpy="0 0 0"/>
         <geometry>
-          <mesh filename="package://onrobot_2fg7_description/meshes/base_link.stl" scale="0.001 0.001 0.001"/>
+          <mesh filename="package://onrobot_2fg7_description/urdf/meshes/base_link.stl" scale="0.001 0.001 0.001"/>
         </geometry>
       </collision>
@@ -38,5 +38,5 @@
         <origin xyz="0.054361 0.029494 -0.12005" rpy="0 0 0"/>
         <geometry>
-          <mesh filename="package://onrobot_2fg7_description/meshes/right_finger_link.stl" scale="0.001 0.001 0.001"/>
+          <mesh filename="package://onrobot_2fg7_description/urdf/meshes/right_finger_link.stl" scale="0.001 0.001 0.001"/>
         </geometry>
         <material name="silver"/>
@@ -45,5 +45,5 @@
         <origin xyz="0.054361 0.029494 -0.12005" rpy="0 0 0"/>
         <geometry>
-          <mesh filename="package://onrobot_2fg7_description/meshes/right_finger_link.stl" scale="0.001 0.001 0.001"/>
+          <mesh filename="package://onrobot_2fg7_description/urdf/meshes/right_finger_link.stl" scale="0.001 0.001 0.001"/>
         </geometry>
       </collision>
@@ -58,5 +58,5 @@
         <origin xyz="-0.032239 0.029494 -0.12005" rpy="0 0 0"/>
         <geometry>
-          <mesh filename="package://onrobot_2fg7_description/meshes/left_finger_link.stl" scale="0.001 0.001 0.001"/>
+          <mesh filename="package://onrobot_2fg7_description/urdf/meshes/left_finger_link.stl" scale="0.001 0.001 0.001"/>
         </geometry>
         <material name="silver"/>
@@ -65,5 +65,5 @@
         <origin xyz="-0.032239 0.029494 -0.12005" rpy="0 0 0"/>
         <geometry>
-          <mesh filename="package://onrobot_2fg7_description/meshes/left_finger_link.stl" scale="0.001 0.001 0.001"/>
+          <mesh filename="package://onrobot_2fg7_description/urdf/meshes/left_finger_link.stl" scale="0.001 0.001 0.001"/>
         </geometry>
       </collision>
@@ -95,5 +95,5 @@
         <origin xyz="0 0 0" rpy="0 0 0"/>
         <geometry>
-          <mesh filename="package://onrobot_2fg7_description/meshes/base_link.stl" scale="0.001 0.001 0.001"/>
+          <mesh filename="package://onrobot_2fg7_description/urdf/meshes/base_link.stl" scale="0.001 0.001 0.001"/>
         </geometry>
         <material name="silver"/>
@@ -102,5 +102,5 @@
         <origin xyz="0 0 0" rpy="0 0 0"/>
         <geometry>
-          <mesh filename="package://onrobot_2fg7_description/meshes/base_link.stl" scale="0.001 0.001 0.001"/>
+          <mesh filename="package://onrobot_2fg7_description/urdf/meshes/base_link.stl" scale="0.001 0.001 0.001"/>
         </geometry>
       </collision>
@@ -115,5 +115,5 @@
         <origin xyz="0.054361 0.029494 -0.12005" rpy="0 0 0"/>
         <geometry>
-          <mesh filename="package://onrobot_2fg7_description/meshes/inwards/right_finger_link.stl" scale="0.001 0.001 0.001"/>
+          <mesh filename="package://onrobot_2fg7_description/urdf/meshes/inwards/right_finger_link.stl" scale="0.001 0.001 0.001"/>
         </geometry>
         <material name="silver"/>
@@ -122,5 +122,5 @@
         <origin xyz="0.054361 0.029494 -0.12005" rpy="0 0 0"/>
         <geometry>
-          <mesh filename="package://onrobot_2fg7_description/meshes/inwards/right_finger_link.stl" scale="0.001 0.001 0.001"/>
+          <mesh filename="package://onrobot_2fg7_description/urdf/meshes/inwards/right_finger_link.stl" scale="0.001 0.001 0.001"/>
         </geometry>
       </collision>
@@ -135,5 +135,5 @@
         <origin xyz="-0.032239 0.029494 -0.12005" rpy="0 0 0"/>
         <geometry>
-          <mesh filename="package://onrobot_2fg7_description/meshes/inwards/left_finger_link.stl" scale="0.001 0.001 0.001"/>
+          <mesh filename="package://onrobot_2fg7_description/urdf/meshes/inwards/left_finger_link.stl" scale="0.001 0.001 0.001"/>
         </geometry>
         <material name="silver"/>
@@ -142,5 +142,5 @@
         <origin xyz="-0.032239 0.029494 -0.12005" rpy="0 0 0"/>
         <geometry>
-          <mesh filename="package://onrobot_2fg7_description/meshes/inwards/left_finger_link.stl" scale="0.001 0.001 0.001"/>
+          <mesh filename="package://onrobot_2fg7_description/urdf/meshes/inwards/left_finger_link.stl" scale="0.001 0.001 0.001"/>
         </geometry>
       </collision>

Commit message: ROS2 migration - Repo Name FIX

File: urdf/onrobot_2fg7.xacro (robot description, xacro)
@@ -1,7 +1,7 @@
 <?xml version="1.0" ?>
 <robot name="2fg7_outwards" xmlns:xacro="http://www.ros.org/wiki/xacro">
-<xacro:include filename="$(find onrobot_2fg7_description)/urdf/materials.xacro" />
-<xacro:include filename="$(find onrobot_2fg7_description)/urdf/onrobot_2fg7.trans.xacro" />
-<xacro:include filename="$(find onrobot_2fg7_description)/urdf/onrobot_2fg7.gazebo" />
+<xacro:include filename="$(find onrobot_2FG7_gripper_description)/urdf/materials.xacro" />
+<xacro:include filename="$(find onrobot_2FG7_gripper_description)/urdf/onrobot_2fg7.trans.xacro" />
+<xacro:include filename="$(find onrobot_2FG7_gripper_description)/urdf/onrobot_2fg7.gazebo" />
 <xacro:gripper_transmission/>
 <xacro:gazebo_control is_control_on="false" />
@@ -18,5 +18,5 @@
         <origin xyz="0 0 0" rpy="0 0 0"/>
         <geometry>
-          <mesh filename="package://onrobot_2fg7_description/urdf/meshes/base_link.stl" scale="0.001 0.001 0.001"/>
+          <mesh filename="package://onrobot_2FG7_gripper_description/urdf/meshes/base_link.stl" scale="0.001 0.001 0.001"/>
         </geometry>
         <material name="silver"/>
@@ -25,5 +25,5 @@
         <origin xyz="0 0 0" rpy="0 0 0"/>
         <geometry>
-          <mesh filename="package://onrobot_2fg7_description/urdf/meshes/base_link.stl" scale="0.001 0.001 0.001"/>
+          <mesh filename="package://onrobot_2FG7_gripper_description/urdf/meshes/base_link.stl" scale="0.001 0.001 0.001"/>
         </geometry>
       </collision>
@@ -38,5 +38,5 @@
         <origin xyz="0.054361 0.029494 -0.12005" rpy="0 0 0"/>
         <geometry>
-          <mesh filename="package://onrobot_2fg7_description/urdf/meshes/right_finger_link.stl" scale="0.001 0.001 0.001"/>
+          <mesh filename="package://onrobot_2FG7_gripper_description/urdf/meshes/right_finger_link.stl" scale="0.001 0.001 0.001"/>
         </geometry>
         <material name="silver"/>
@@ -45,5 +45,5 @@
         <origin xyz="0.054361 0.029494 -0.12005" rpy="0 0 0"/>
         <geometry>
-          <mesh filename="package://onrobot_2fg7_description/urdf/meshes/right_finger_link.stl" scale="0.001 0.001 0.001"/>
+          <mesh filename="package://onrobot_2FG7_gripper_description/urdf/meshes/right_finger_link.stl" scale="0.001 0.001 0.001"/>
         </geometry>
       </collision>
@@ -58,5 +58,5 @@
         <origin xyz="-0.032239 0.029494 -0.12005" rpy="0 0 0"/>
         <geometry>
-          <mesh filename="package://onrobot_2fg7_description/urdf/meshes/left_finger_link.stl" scale="0.001 0.001 0.001"/>
+          <mesh filename="package://onrobot_2FG7_gripper_description/urdf/meshes/left_finger_link.stl" scale="0.001 0.001 0.001"/>
         </geometry>
         <material name="silver"/>
@@ -65,5 +65,5 @@
         <origin xyz="-0.032239 0.029494 -0.12005" rpy="0 0 0"/>
         <geometry>
-          <mesh filename="package://onrobot_2fg7_description/urdf/meshes/left_finger_link.stl" scale="0.001 0.001 0.001"/>
+          <mesh filename="package://onrobot_2FG7_gripper_description/urdf/meshes/left_finger_link.stl" scale="0.001 0.001 0.001"/>
         </geometry>
       </collision>
@@ -95,5 +95,5 @@
         <origin xyz="0 0 0" rpy="0 0 0"/>
         <geometry>
-          <mesh filename="package://onrobot_2fg7_description/urdf/meshes/base_link.stl" scale="0.001 0.001 0.001"/>
+          <mesh filename="package://onrobot_2FG7_gripper_description/urdf/meshes/base_link.stl" scale="0.001 0.001 0.001"/>
         </geometry>
         <material name="silver"/>
@@ -102,5 +102,5 @@
         <origin xyz="0 0 0" rpy="0 0 0"/>
         <geometry>
-          <mesh filename="package://onrobot_2fg7_description/urdf/meshes/base_link.stl" scale="0.001 0.001 0.001"/>
+          <mesh filename="package://onrobot_2FG7_gripper_description/urdf/meshes/base_link.stl" scale="0.001 0.001 0.001"/>
         </geometry>
       </collision>
@@ -115,5 +115,5 @@
         <origin xyz="0.054361 0.029494 -0.12005" rpy="0 0 0"/>
         <geometry>
-          <mesh filename="package://onrobot_2fg7_description/urdf/meshes/inwards/right_finger_link.stl" scale="0.001 0.001 0.001"/>
+          <mesh filename="package://onrobot_2FG7_gripper_description/urdf/meshes/inwards/right_finger_link.stl" scale="0.001 0.001 0.001"/>
         </geometry>
         <material name="silver"/>
@@ -122,5 +122,5 @@
         <origin xyz="0.054361 0.029494 -0.12005" rpy="0 0 0"/>
         <geometry>
-          <mesh filename="package://onrobot_2fg7_description/urdf/meshes/inwards/right_finger_link.stl" scale="0.001 0.001 0.001"/>
+          <mesh filename="package://onrobot_2FG7_gripper_description/urdf/meshes/inwards/right_finger_link.stl" scale="0.001 0.001 0.001"/>
         </geometry>
       </collision>
@@ -135,5 +135,5 @@
         <origin xyz="-0.032239 0.029494 -0.12005" rpy="0 0 0"/>
         <geometry>
-          <mesh filename="package://onrobot_2fg7_description/urdf/meshes/inwards/left_finger_link.stl" scale="0.001 0.001 0.001"/>
+          <mesh filename="package://onrobot_2FG7_gripper_description/urdf/meshes/inwards/left_finger_link.stl" scale="0.001 0.001 0.001"/>
         </geometry>
         <material name="silver"/>
@@ -142,5 +142,5 @@
         <origin xyz="-0.032239 0.029494 -0.12005" rpy="0 0 0"/>
         <geometry>
-          <mesh filename="package://onrobot_2fg7_description/urdf/meshes/inwards/left_finger_link.stl" scale="0.001 0.001 0.001"/>
+          <mesh filename="package://onrobot_2FG7_gripper_description/urdf/meshes/inwards/left_finger_link.stl" scale="0.001 0.001 0.001"/>
         </geometry>
       </collision>

File: urdf/onrobot_2fg7_upload.xacro (robot description, xacro)
@@ -1,5 +1,5 @@
 <?xml version="1.0" ?>
 <robot name="2fg7_outwards" xmlns:xacro="http://www.ros.org/wiki/xacro">
-  <xacro:include filename="$(find onrobot_2fg7_description)/urdf/onrobot_2fg7.xacro" />
+  <xacro:include filename="$(find onrobot_2FG7_gripper_description)/urdf/onrobot_2fg7.xacro" />
  <xacro:onrobot_2fg7_gripper prefix="" finger_configuration="outwards"/>
   <link name="world" />
@@ -9,6 +9,6 @@
     <origin xyz="0.0 0.0 0.0" rpy="0.0 0.0 0.0" />
   </joint>
-  <xacro:include filename="$(find onrobot_2fg7_description)/urdf/gzplugin_grasp_fix.urdf.xacro"/>
-  <xacro:include filename="$(find onrobot_2fg7_description)/urdf/mimic_fix.urdf.xacro"/>
+  <xacro:include filename="$(find onrobot_2FG7_gripper_description)/urdf/gzplugin_grasp_fix.urdf.xacro"/>
+  <xacro:include filename="$(find onrobot_2FG7_gripper_description)/urdf/mimic_fix.urdf.xacro"/>
   <xacro:gzplugin_grasp_fix/>
   <xacro:mimic_fix/>
