Commit message: xacro upload

File: urdf/onrobot_2fg7.xacro (robot description, xacro)
@@ -1,166 +1,165 @@
 <?xml version="1.0" ?>
 <robot name="2fg7_outwards" xmlns:xacro="http://www.ros.org/wiki/xacro">
-<xacro:include filename="$(find onrobot_2fg7_gripper_description)/urdf/materials.xacro" />
-<xacro:include filename="$(find onrobot_2fg7_gripper_description)/urdf/onrobot_2fg7.trans.xacro" />
-<xacro:include filename="$(find onrobot_2fg7_gripper_description)/urdf/onrobot_2fg7.gazebo" />
-<xacro:gripper_transmission/>
-<xacro:gazebo_control is_control_on="false" />
+  <xacro:include filename="$(find onrobot_2fg7_gripper_description)/urdf/materials.xacro" />
+  <xacro:include filename="$(find onrobot_2fg7_gripper_description)/urdf/onrobot_2fg7.trans.xacro" />
+  <xacro:include filename="$(find onrobot_2fg7_gripper_description)/urdf/onrobot_2fg7.gazebo" />
+  <xacro:gripper_transmission/>
+  <xacro:gazebo_control is_control_on="false" />
+  <xacro:macro name="onrobot_2fg7_gripper" params="prefix finger_configuration=outwards">
+    <xacro:property name="config" value="${finger_configuration}"/>
+    <xacro:if value="${config == 'outwards'}">
+      <link name="${prefix}base_link">
+        <inertial>
+          <origin xyz="-4.898915958379213e-05 2.84756960271082e-06 0.06811082379774974" rpy="0 0 0"/>
+          <mass value="1.2646523179240972"/>
+          <inertia ixx="0.001504" iyy="0.001812" izz="0.001053" ixy="-0.0" iyz="0.0" ixz="-3e-06"/>
+        </inertial>
+        <visual>
+          <origin xyz="0 0 0" rpy="0 0 0"/>
+          <geometry>
+            <mesh filename="package://onrobot_2fg7_gripper_description/meshes/base_link.stl" scale="0.001 0.001 0.001"/>
+          </geometry>
+          <material name="silver"/>
+        </visual>
+        <collision>
+          <origin xyz="0 0 0" rpy="0 0 0"/>
+          <geometry>
+            <mesh filename="package://onrobot_2fg7_gripper_description/meshes/base_link.stl" scale="0.001 0.001 0.001"/>
+          </geometry>
+        </collision>
+      </link>
+      <link name="${prefix}right_finger_link">
+        <inertial>
+          <origin xyz="0.017874296677847158 0.02949104051991925 0.01523421548622829" rpy="0 0 0"/>
+          <mass value="0.023219383355922288"/>
+          <inertia ixx="6e-06" iyy="5e-06" izz="2e-06" ixy="-0.0" iyz="-0.0" ixz="1e-06"/>
+        </inertial>
+        <visual>
+          <origin xyz="0.054361 0.029494 -0.12005" rpy="0 0 0"/>
+          <geometry>
+            <mesh filename="package://onrobot_2fg7_gripper_description/meshes/right_finger_link.stl" scale="0.001 0.001 0.001"/>
+          </geometry>
+          <material name="silver"/>
+        </visual>
+        <collision name="right_finger_collision">
+          <origin xyz="0.054361 0.029494 -0.12005" rpy="0 0 0"/>
+          <geometry>
+            <mesh filename="package://onrobot_2fg7_gripper_description/meshes/right_finger_link.stl" scale="0.001 0.001 0.001"/>
+          </geometry>
+        </collision>
+      </link>
+      <link name="${prefix}left_finger_link">
+        <inertial>
+          <origin xyz="0.004247703322119739 0.029496959480080673 0.015234215486237948" rpy="0 0 0"/>
+          <mass value="0.023219383355922288"/>
+          <inertia ixx="6e-06" iyy="5e-06" izz="2e-06" ixy="-0.0" iyz="0.0" ixz="-1e-06"/>
+        </inertial>
+        <visual>
+          <origin xyz="-0.032239 0.029494 -0.12005" rpy="0 0 0"/>
+          <geometry>
+            <mesh filename="package://onrobot_2fg7_gripper_description/meshes/left_finger_link.stl" scale="0.001 0.001 0.001"/>
+          </geometry>
+          <material name="silver"/>
+        </visual>
+        <collision name="left_finger_collision">
+          <origin xyz="-0.032239 0.029494 -0.12005" rpy="0 0 0"/>
+          <geometry>
+            <mesh filename="package://onrobot_2fg7_gripper_description/meshes/left_finger_link.stl" scale="0.001 0.001 0.001"/>
+          </geometry>
+        </collision>
+      </link>
+      <joint name="left_finger_joint" type="prismatic">
+        <origin xyz="0.032239 -0.029494 0.12005" rpy="0 0 0"/>
+        <parent link="${prefix}base_link"/>
+        <child link="${prefix}left_finger_link"/>
+        <axis xyz="-1.0 0.0 0.0"/>
+        <limit lower="0.0" upper="0.019" effort="140" velocity="0.45"/> <!-- total 0.38 -->
+      </joint>
+      <joint name="right_finger_joint" type="prismatic">
+        <origin xyz="-0.054361 -0.029494 0.12005" rpy="0 0 0"/>
+        <parent link="${prefix}base_link"/>
+        <child link="${prefix}right_finger_link"/>
+        <axis xyz="1.0 0.0 0.0"/>
+        <limit lower="-0.019" upper="0.019" effort="140" velocity="0.45"/>
+        <mimic joint="left_finger_joint" multiplier="1.0"/>
+      </joint>
+    </xacro:if>
+    <xacro:if value="${config == 'inwards'}">
+      <link name="${prefix}base_link">
+        <inertial>
+          <origin xyz="-4.8989159583623376e-05 2.847569602502098e-06 0.06811082379775064" rpy="0 0 0"/>
+          <mass value="1.2646523179240972"/>
+          <inertia ixx="0.001504" iyy="0.001812" izz="0.001053" ixy="-0.0" iyz="0.0" ixz="-3e-06"/>
+        </inertial>
+        <visual>
+          <origin xyz="0 0 0" rpy="0 0 0"/>
+          <geometry>
+            <mesh filename="package://onrobot_2fg7_gripper_description/meshes/base_link.stl" scale="0.001 0.001 0.001"/>
+          </geometry>
+          <material name="silver"/>
+        </visual>
+        <collision>
+          <origin xyz="0 0 0" rpy="0 0 0"/>
+          <geometry>
+            <mesh filename="package://onrobot_2fg7_gripper_description/meshes/base_link.stl" scale="0.001 0.001 0.001"/>
+          </geometry>
+        </collision>
+      </link>
+      <link name="${prefix}right_finger_link">
+        <inertial>
+          <origin xyz="0.029847703322119633 0.029496959480087837 0.015234215486232036" rpy="0 0 0"/>
+          <mass value="0.023219383355922288"/>
+          <inertia ixx="6e-06" iyy="5e-06" izz="2e-06" ixy="-0.0" iyz="0.0" ixz="-1e-06"/>
+        </inertial>
+        <visual>
+          <origin xyz="0.054361 0.029494 -0.12005" rpy="0 0 0"/>
+          <geometry>
+            <mesh filename="package://onrobot_2fg7_gripper_description/meshes/inwards/right_finger_link.stl" scale="0.001 0.001 0.001"/>
+          </geometry>
+          <material name="silver"/>
+        </visual>
+        <collision>
+          <origin xyz="0.054361 0.029494 -0.12005" rpy="0 0 0"/>
+          <geometry>
+            <mesh filename="package://onrobot_2fg7_gripper_description/meshes/inwards/right_finger_link.stl" scale="0.001 0.001 0.001"/>
+          </geometry>
+        </collision>
+      </link>
+      <link name="${prefix}left_finger_link">
+        <inertial>
+          <origin xyz="-0.007725703322151688 0.029491040519911117 0.015234215486238503" rpy="0 0 0"/>
+          <mass value="0.023219383355922288"/>
+          <inertia ixx="6e-06" iyy="5e-06" izz="2e-06" ixy="-0.0" iyz="-0.0" ixz="1e-06"/>
+        </inertial>
+        <visual>
+          <origin xyz="-0.032239 0.029494 -0.12005" rpy="0 0 0"/>
+          <geometry>
+            <mesh filename="package://onrobot_2fg7_gripper_description/meshes/inwards/left_finger_link.stl" scale="0.001 0.001 0.001"/>
+          </geometry>
+          <material name="silver"/>
+        </visual>
+        <collision>
+          <origin xyz="-0.032239 0.029494 -0.12005" rpy="0 0 0"/>
+          <geometry>
+            <mesh filename="package://onrobot_2fg7_gripper_description/meshes/inwards/left_finger_link.stl" scale="0.001 0.001 0.001"/>
+          </geometry>
+        </collision>
+      </link>
+      <joint name="left_finger_joint" type="prismatic">
+        <origin xyz="0.032239 -0.029494 0.12005" rpy="0 0 0"/>
+        <parent link="${prefix}base_link"/>
+        <child link="${prefix}left_finger_link"/>
+        <axis xyz="-1.0 0.0 0.0"/>
+        <limit upper="0.0" lower="0.019" effort="100" velocity="0.45"/>
+      </joint>
+      <joint name="right_finger_joint" type="prismatic">
+        <origin xyz="-0.054361 -0.029494 0.12005" rpy="0 0 0"/>
+        <parent link="${prefix}base_link"/>
+        <child link="${prefix}right_finger_link"/>
+        <axis xyz="1.0 0.0 0.0"/>
+        <limit lower="-0.019" upper="0.019" effort="100" velocity="0.45"/>
+        <mimic joint="left_finger_joint" multiplier="1.0"/>
+      </joint>
+    </xacro:if>
+  </xacro:macro>
 </robot>
-<xacro:macro name="onrobot_2fg7_gripper" params="prefix finger_configuration=outwards">
-  <xacro:property name="config" value="${finger_configuration}"/>
-  <xacro:if value="${config == 'outwards'}">
-    <link name="${prefix}base_link">
-      <inertial>
-        <origin xyz="-4.898915958379213e-05 2.84756960271082e-06 0.06811082379774974" rpy="0 0 0"/>
-        <mass value="1.2646523179240972"/>
-        <inertia ixx="0.001504" iyy="0.001812" izz="0.001053" ixy="-0.0" iyz="0.0" ixz="-3e-06"/>
-      </inertial>
-      <visual>
-        <origin xyz="0 0 0" rpy="0 0 0"/>
-        <geometry>
-          <mesh filename="package://onrobot_2fg7_gripper_description/meshes/base_link.stl" scale="0.001 0.001 0.001"/>
-        </geometry>
-        <material name="silver"/>
-      </visual>
-      <collision>
-        <origin xyz="0 0 0" rpy="0 0 0"/>
-        <geometry>
-          <mesh filename="package://onrobot_2fg7_gripper_description/meshes/base_link.stl" scale="0.001 0.001 0.001"/>
-        </geometry>
-      </collision>
-    </link>
-    <link name="${prefix}right_finger_link">
-      <inertial>
-        <origin xyz="0.017874296677847158 0.02949104051991925 0.01523421548622829" rpy="0 0 0"/>
-        <mass value="0.023219383355922288"/>
-        <inertia ixx="6e-06" iyy="5e-06" izz="2e-06" ixy="-0.0" iyz="-0.0" ixz="1e-06"/>
-      </inertial>
-      <visual>
-        <origin xyz="0.054361 0.029494 -0.12005" rpy="0 0 0"/>
-        <geometry>
-          <mesh filename="package://onrobot_2fg7_gripper_description/meshes/right_finger_link.stl" scale="0.001 0.001 0.001"/>
-        </geometry>
-        <material name="silver"/>
-      </visual>
-      <collision name="right_finger_collision">
-        <origin xyz="0.054361 0.029494 -0.12005" rpy="0 0 0"/>
-        <geometry>
-          <mesh filename="package://onrobot_2fg7_gripper_description/meshes/right_finger_link.stl" scale="0.001 0.001 0.001"/>
-        </geometry>
-      </collision>
-    </link>
-    <link name="${prefix}left_finger_link">
-      <inertial>
-        <origin xyz="0.004247703322119739 0.029496959480080673 0.015234215486237948" rpy="0 0 0"/>
-        <mass value="0.023219383355922288"/>
-        <inertia ixx="6e-06" iyy="5e-06" izz="2e-06" ixy="-0.0" iyz="0.0" ixz="-1e-06"/>
-      </inertial>
-      <visual>
-        <origin xyz="-0.032239 0.029494 -0.12005" rpy="0 0 0"/>
-        <geometry>
-          <mesh filename="package://onrobot_2fg7_gripper_description/meshes/left_finger_link.stl" scale="0.001 0.001 0.001"/>
-        </geometry>
-        <material name="silver"/>
-      </visual>
-      <collision name="left_finger_collision">
-        <origin xyz="-0.032239 0.029494 -0.12005" rpy="0 0 0"/>
-        <geometry>
-          <mesh filename="package://onrobot_2fg7_gripper_description/meshes/left_finger_link.stl" scale="0.001 0.001 0.001"/>
-        </geometry>
-      </collision>
-    </link>
-    <joint name="left_finger_joint" type="prismatic">
-      <origin xyz="0.032239 -0.029494 0.12005" rpy="0 0 0"/>
-      <parent link="${prefix}base_link"/>
-      <child link="${prefix}left_finger_link"/>
-      <axis xyz="-1.0 0.0 0.0"/>
-      <limit lower="0.0" upper="0.019" effort="140" velocity="0.45"/> <!-- total 0.38 -->
-    </joint>
-    <joint name="right_finger_joint" type="prismatic">
-      <origin xyz="-0.054361 -0.029494 0.12005" rpy="0 0 0"/>
-      <parent link="${prefix}base_link"/>
-      <child link="${prefix}right_finger_link"/>
-      <axis xyz="1.0 0.0 0.0"/>
-      <limit lower="-0.019" upper="0.019" effort="140" velocity="0.45"/>
-      <mimic joint="left_finger_joint" multiplier="1.0"/>
-    </joint>
-  </xacro:if>
-   <xacro:if value="${config == 'inwards'}">
-    <link name="${prefix}base_link">
-      <inertial>
-        <origin xyz="-4.8989159583623376e-05 2.847569602502098e-06 0.06811082379775064" rpy="0 0 0"/>
-        <mass value="1.2646523179240972"/>
-        <inertia ixx="0.001504" iyy="0.001812" izz="0.001053" ixy="-0.0" iyz="0.0" ixz="-3e-06"/>
-      </inertial>
-      <visual>
-        <origin xyz="0 0 0" rpy="0 0 0"/>
-        <geometry>
-          <mesh filename="package://onrobot_2fg7_gripper_description/meshes/base_link.stl" scale="0.001 0.001 0.001"/>
-        </geometry>
-        <material name="silver"/>
-      </visual>
-      <collision>
-        <origin xyz="0 0 0" rpy="0 0 0"/>
-        <geometry>
-          <mesh filename="package://onrobot_2fg7_gripper_description/meshes/base_link.stl" scale="0.001 0.001 0.001"/>
-        </geometry>
-      </collision>
-    </link>
-    <link name="${prefix}right_finger_link">
-      <inertial>
-        <origin xyz="0.029847703322119633 0.029496959480087837 0.015234215486232036" rpy="0 0 0"/>
-        <mass value="0.023219383355922288"/>
-        <inertia ixx="6e-06" iyy="5e-06" izz="2e-06" ixy="-0.0" iyz="0.0" ixz="-1e-06"/>
-      </inertial>
-      <visual>
-        <origin xyz="0.054361 0.029494 -0.12005" rpy="0 0 0"/>
-        <geometry>
-          <mesh filename="package://onrobot_2fg7_gripper_description/meshes/inwards/right_finger_link.stl" scale="0.001 0.001 0.001"/>
-        </geometry>
-        <material name="silver"/>
-      </visual>
-      <collision>
-        <origin xyz="0.054361 0.029494 -0.12005" rpy="0 0 0"/>
-        <geometry>
-          <mesh filename="package://onrobot_2fg7_gripper_description/meshes/inwards/right_finger_link.stl" scale="0.001 0.001 0.001"/>
-        </geometry>
-      </collision>
-    </link>
-    <link name="${prefix}left_finger_link">
-      <inertial>
-        <origin xyz="-0.007725703322151688 0.029491040519911117 0.015234215486238503" rpy="0 0 0"/>
-        <mass value="0.023219383355922288"/>
-        <inertia ixx="6e-06" iyy="5e-06" izz="2e-06" ixy="-0.0" iyz="-0.0" ixz="1e-06"/>
-      </inertial>
-      <visual>
-        <origin xyz="-0.032239 0.029494 -0.12005" rpy="0 0 0"/>
-        <geometry>
-          <mesh filename="package://onrobot_2fg7_gripper_description/meshes/inwards/left_finger_link.stl" scale="0.001 0.001 0.001"/>
-        </geometry>
-        <material name="silver"/>
-      </visual>
-      <collision>
-        <origin xyz="-0.032239 0.029494 -0.12005" rpy="0 0 0"/>
-        <geometry>
-          <mesh filename="package://onrobot_2fg7_gripper_description/meshes/inwards/left_finger_link.stl" scale="0.001 0.001 0.001"/>
-        </geometry>
-      </collision>
-    </link>
-    <joint name="left_finger_joint" type="prismatic">
-      <origin xyz="0.032239 -0.029494 0.12005" rpy="0 0 0"/>
-      <parent link="${prefix}base_link"/>
-      <child link="${prefix}left_finger_link"/>
-      <axis xyz="-1.0 0.0 0.0"/>
-      <limit upper="0.0" lower="0.019" effort="100" velocity="0.45"/>
-    </joint>
-    <joint name="right_finger_joint" type="prismatic">
-      <origin xyz="-0.054361 -0.029494 0.12005" rpy="0 0 0"/>
-      <parent link="${prefix}base_link"/>
-      <child link="${prefix}right_finger_link"/>
-      <axis xyz="1.0 0.0 0.0"/>
-      <limit lower="-0.019" upper="0.019" effort="100" velocity="0.45"/>
-      <mimic joint="left_finger_joint" multiplier="1.0"/>
-    </joint>
-   </xacro:if>
- </xacro:macro>
-</robot>

Commit message: firx try6

File: urdf/onrobot_2fg7.xacro (robot description, xacro)
@@ -4,5 +4,5 @@
   <xacro:include filename="$(find onrobot_2fg7_gripper_description)/urdf/onrobot_2fg7.trans.xacro" />
   <xacro:include filename="$(find onrobot_2fg7_gripper_description)/urdf/onrobot_2fg7.gazebo" />
-  <xacro:macro name="onrobot_2fg7_gripper" params="prefix finger_configuration=outwards">
+  <xacro:macro name="onrobot_2fg7_gripper" params="parent prefix finger_configuration=outwards">
     <xacro:gripper_transmission/>
     <xacro:gazebo_control is_control_on="false" />

Commit message: firx try7

File: urdf/onrobot_2fg7.xacro (robot description, xacro)
@@ -5,4 +5,10 @@
   <xacro:include filename="$(find onrobot_2fg7_gripper_description)/urdf/onrobot_2fg7.gazebo" />
   <xacro:macro name="onrobot_2fg7_gripper" params="parent prefix finger_configuration=outwards">
+    <!-- CRITICAL FIX: Add joint to connect gripper base to parent link -->
+    <joint name="${prefix}base_joint" type="fixed">
+      <parent link="${parent}"/>
+      <child link="${prefix}base_link"/>
+      <origin xyz="0 0 0" rpy="0 0 0"/>
+    </joint>
     <xacro:gripper_transmission/>
     <xacro:gazebo_control is_control_on="false" />

Commit message: Joint limits fix

File: urdf/onrobot_2fg7.xacro (robot description, xacro)
@@ -152,4 +152,5 @@
         </collision>
       </link>
+      <!-- CORRECTED limits for 2FG7 gripper -->
       <joint name="left_finger_joint" type="prismatic">
         <origin xyz="0.032239 -0.029494 0.12005" rpy="0 0 0"/>
@@ -157,5 +158,6 @@
         <child link="${prefix}left_finger_link"/>
         <axis xyz="-1.0 0.0 0.0"/>
-        <limit upper="0.0" lower="0.019" effort="100" velocity="0.45"/>
+        <!-- FIX: Each finger moves 20mm from center (35mm to 75mm total) -->
+        <limit lower="0.0" upper="0.020" effort="100" velocity="0.45"/>
       </joint>
       <joint name="right_finger_joint" type="prismatic">
@@ -164,5 +166,6 @@
         <child link="${prefix}right_finger_link"/>
         <axis xyz="1.0 0.0 0.0"/>
-        <limit lower="-0.019" upper="0.019" effort="100" velocity="0.45"/>
+        <!-- FIX: Mirror the left finger -->
+        <limit lower="-0.020" upper="0.0" effort="100" velocity="0.45"/>
         <mimic joint="left_finger_joint" multiplier="1.0"/>
       </joint>

Commit message: Joint limits fix 2

File: urdf/onrobot_2fg7.xacro (robot description, xacro)
@@ -159,5 +159,5 @@
         <axis xyz="-1.0 0.0 0.0"/>
         <!-- FIX: Each finger moves 20mm from center (35mm to 75mm total) -->
-        <limit lower="0.0" upper="0.020" effort="100" velocity="0.45"/>
+        <limit lower="0.0175" upper="0.0375" effort="100" velocity="0.45"/>
       </joint>
       <joint name="right_finger_joint" type="prismatic">
@@ -167,5 +167,5 @@
         <axis xyz="1.0 0.0 0.0"/>
         <!-- FIX: Mirror the left finger -->
-        <limit lower="-0.020" upper="0.0" effort="100" velocity="0.45"/>
+        <limit lower="-0.0375" upper="-0.0175" effort="100" velocity="0.45"/>
         <mimic joint="left_finger_joint" multiplier="1.0"/>
       </joint>

Commit message: Joint limits fix attempt 2 - try 1

File: urdf/onrobot_2fg7.xacro (robot description, xacro)
@@ -154,5 +154,5 @@
       <!-- CORRECTED limits for 2FG7 gripper -->
       <joint name="left_finger_joint" type="prismatic">
-        <origin xyz="0.032239 -0.029494 0.12005" rpy="0 0 0"/>
+        <origin xyz="0.035 -0.029494 0.12005" rpy="0 0 0"/>
         <parent link="${prefix}base_link"/>
         <child link="${prefix}left_finger_link"/>
@@ -162,5 +162,5 @@
       </joint>
       <joint name="right_finger_joint" type="prismatic">
-        <origin xyz="-0.054361 -0.029494 0.12005" rpy="0 0 0"/>
+        <origin xyz="-0.035 -0.029494 0.12005" rpy="0 0 0"/>
         <parent link="${prefix}base_link"/>
         <child link="${prefix}right_finger_link"/>

Commit message: Fix Joint Limits for 75mm-35mm Gripper

File: urdf/onrobot_2fg7.xacro (robot description, xacro)
@@ -152,20 +152,20 @@
         </collision>
       </link>
-      <!-- CORRECTED limits for 2FG7 gripper -->
+      <!-- For outward configuration -->
       <joint name="left_finger_joint" type="prismatic">
-        <origin xyz="0.035 -0.029494 0.12005" rpy="0 0 0"/>
+        <origin xyz="0.032239 -0.029494 0.12005" rpy="0 0 0"/>
         <parent link="${prefix}base_link"/>
         <child link="${prefix}left_finger_link"/>
         <axis xyz="-1.0 0.0 0.0"/>
-        <!-- FIX: Each finger moves 20mm from center (35mm to 75mm total) -->
-        <limit lower="0.0175" upper="0.0375" effort="100" velocity="0.45"/>
+        <!-- CORRECTED: Each finger moves 20mm from center (35mm to 75mm total) -->
+        <limit lower="0.0" upper="0.020" effort="140" velocity="0.45"/>
       </joint>
       <joint name="right_finger_joint" type="prismatic">
-        <origin xyz="-0.035 -0.029494 0.12005" rpy="0 0 0"/>
+        <origin xyz="-0.054361 -0.029494 0.12005" rpy="0 0 0"/>
         <parent link="${prefix}base_link"/>
         <child link="${prefix}right_finger_link"/>
         <axis xyz="1.0 0.0 0.0"/>
-        <!-- FIX: Mirror the left finger -->
-        <limit lower="-0.0375" upper="-0.0175" effort="100" velocity="0.45"/>
+        <!-- CORRECTED: Mirror the left finger -->
+        <limit lower="-0.020" upper="0.0" effort="140" velocity="0.45"/>
         <mimic joint="left_finger_joint" multiplier="1.0"/>
       </joint>
