Commit message: removing large offsets

File: urdf/onrobot_2fg7.xacro (robot description, xacro)
@@ -42,5 +42,6 @@
         </inertial>
         <visual>
-          <origin xyz="0.054361 0.029494 -0.12005" rpy="0 0 0"/>
+          <!-- FIXED: Remove large offset from visual origin -->
+          <origin xyz="0 0 0" rpy="0 0 0"/>
           <geometry>
             <mesh filename="package://onrobot_2fg7_gripper_description/meshes/right_finger_link.stl" scale="0.001 0.001 0.001"/>
@@ -49,5 +50,6 @@
         </visual>
         <collision name="right_finger_collision">
-          <origin xyz="0.054361 0.029494 -0.12005" rpy="0 0 0"/>
+          <!-- FIXED: Remove large offset from collision origin -->
+          <origin xyz="0 0 0" rpy="0 0 0"/>
           <geometry>
             <mesh filename="package://onrobot_2fg7_gripper_description/meshes/right_finger_link.stl" scale="0.001 0.001 0.001"/>
@@ -62,5 +64,6 @@
         </inertial>
         <visual>
-          <origin xyz="-0.032239 0.029494 -0.12005" rpy="0 0 0"/>
+          <!-- FIXED: Remove large offset from visual origin -->
+          <origin xyz="0 0 0" rpy="0 0 0"/>
           <geometry>
             <mesh filename="package://onrobot_2fg7_gripper_description/meshes/left_finger_link.stl" scale="0.001 0.001 0.001"/>
@@ -69,5 +72,6 @@
         </visual>
         <collision name="left_finger_collision">
-          <origin xyz="-0.032239 0.029494 -0.12005" rpy="0 0 0"/>
+          <!-- FIXED: Remove large offset from collision origin -->
+          <origin xyz="0 0 0" rpy="0 0 0"/>
           <geometry>
             <mesh filename="package://onrobot_2fg7_gripper_description/meshes/left_finger_link.stl" scale="0.001 0.001 0.001"/>
@@ -75,96 +79,17 @@
         </collision>
       </link>
+      <!-- FIXED: Joint origins positioned correctly relative to base -->
       <joint name="left_finger_joint" type="prismatic">
-        <origin xyz="0.032239 -0.029494 0.12005" rpy="0 0 0"/>
+        <origin xyz="0.032 0.0 0.0" rpy="0 0 0"/>
         <parent link="${prefix}base_link"/>
         <child link="${prefix}left_finger_link"/>
         <axis xyz="-1.0 0.0 0.0"/>
-        <limit lower="0.0" upper="0.019" effort="140" velocity="0.45"/> <!-- total 0.38 -->
+        <limit lower="0.0" upper="0.020" effort="140" velocity="0.45"/>
       </joint>
       <joint name="right_finger_joint" type="prismatic">
-        <origin xyz="-0.054361 -0.029494 0.12005" rpy="0 0 0"/>
+        <origin xyz="-0.032 0.0 0.0" rpy="0 0 0"/>
         <parent link="${prefix}base_link"/>
         <child link="${prefix}right_finger_link"/>
         <axis xyz="1.0 0.0 0.0"/>
-        <limit lower="-0.019" upper="0.019" effort="140" velocity="0.45"/>
-        <mimic joint="left_finger_joint" multiplier="1.0"/>
-      </joint>
-    </xacro:if>
-    <xacro:if value="${config == 'inwards'}">
-      <link name="${prefix}base_link">
-        <inertial>
-          <origin xyz="-4.8989159583623376e-05 2.847569602502098e-06 0.06811082379775064" rpy="0 0 0"/>
-          <mass value="1.2646523179240972"/>
-          <inertia ixx="0.001504" iyy="0.001812" izz="0.001053" ixy="-0.0" iyz="0.0" ixz="-3e-06"/>
-        </inertial>
-        <visual>
-          <origin xyz="0 0 0" rpy="0 0 0"/>
-          <geometry>
-            <mesh filename="package://onrobot_2fg7_gripper_description/meshes/base_link.stl" scale="0.001 0.001 0.001"/>
-          </geometry>
-          <material name="silver"/>
-        </visual>
-        <collision>
-          <origin xyz="0 0 0" rpy="0 0 0"/>
-          <geometry>
-            <mesh filename="package://onrobot_2fg7_gripper_description/meshes/base_link.stl" scale="0.001 0.001 0.001"/>
-          </geometry>
-        </collision>
-      </link>
-      <link name="${prefix}right_finger_link">
-        <inertial>
-          <origin xyz="0.029847703322119633 0.029496959480087837 0.015234215486232036" rpy="0 0 0"/>
-          <mass value="0.023219383355922288"/>
-          <inertia ixx="6e-06" iyy="5e-06" izz="2e-06" ixy="-0.0" iyz="0.0" ixz="-1e-06"/>
-        </inertial>
-        <visual>
-          <origin xyz="0.054361 0.029494 -0.12005" rpy="0 0 0"/>
-          <geometry>
-            <mesh filename="package://onrobot_2fg7_gripper_description/meshes/inwards/right_finger_link.stl" scale="0.001 0.001 0.001"/>
-          </geometry>
-          <material name="silver"/>
-        </visual>
-        <collision>
-          <origin xyz="0.054361 0.029494 -0.12005" rpy="0 0 0"/>
-          <geometry>
-            <mesh filename="package://onrobot_2fg7_gripper_description/meshes/inwards/right_finger_link.stl" scale="0.001 0.001 0.001"/>
-          </geometry>
-        </collision>
-      </link>
-      <link name="${prefix}left_finger_link">
-        <inertial>
-          <origin xyz="-0.007725703322151688 0.029491040519911117 0.015234215486238503" rpy="0 0 0"/>
-          <mass value="0.023219383355922288"/>
-          <inertia ixx="6e-06" iyy="5e-06" izz="2e-06" ixy="-0.0" iyz="-0.0" ixz="1e-06"/>
-        </inertial>
-        <visual>
-          <origin xyz="-0.032239 0.029494 -0.12005" rpy="0 0 0"/>
-          <geometry>
-            <mesh filename="package://onrobot_2fg7_gripper_description/meshes/inwards/left_finger_link.stl" scale="0.001 0.001 0.001"/>
-          </geometry>
-          <material name="silver"/>
-        </visual>
-        <collision>
-          <origin xyz="-0.032239 0.029494 -0.12005" rpy="0 0 0"/>
-          <geometry>
-            <mesh filename="package://onrobot_2fg7_gripper_description/meshes/inwards/left_finger_link.stl" scale="0.001 0.001 0.001"/>
-          </geometry>
-        </collision>
-      </link>
-      <!-- For outward configuration -->
-      <joint name="left_finger_joint" type="prismatic">
-        <origin xyz="0.032239 -0.029494 0.12005" rpy="0 0 0"/>
-        <parent link="${prefix}base_link"/>
-        <child link="${prefix}left_finger_link"/>
-        <axis xyz="-1.0 0.0 0.0"/>
-        <!-- CORRECTED: 0mm to 20mm per finger (35mm to 75mm total opening) -->
-        <limit lower="0.0" upper="0.020" effort="140" velocity="0.45"/>
-      </joint>
-      <joint name="right_finger_joint" type="prismatic">
-        <origin xyz="-0.054361 -0.029494 0.12005" rpy="0 0 0"/>
-        <parent link="${prefix}base_link"/>
-        <child link="${prefix}right_finger_link"/>
-        <axis xyz="1.0 0.0 0.0"/>
-        <!-- CORRECTED: -20mm to 0mm per finger (mirror of left finger) -->
         <limit lower="-0.020" upper="0.0" effort="140" velocity="0.45"/>
         <mimic joint="left_finger_joint" multiplier="1.0"/>

Commit message: version with offsets, but visual origins fixed

File: urdf/onrobot_2fg7.xacro (robot description, xacro)
@@ -42,5 +42,5 @@
         </inertial>
         <visual>
-          <!-- FIXED: Remove large offset from visual origin -->
+          <!-- FIXED: Simplified visual origin - let joint handle positioning -->
           <origin xyz="0 0 0" rpy="0 0 0"/>
           <geometry>
@@ -50,5 +50,5 @@
         </visual>
         <collision name="right_finger_collision">
-          <!-- FIXED: Remove large offset from collision origin -->
+          <!-- FIXED: Simplified collision origin -->
           <origin xyz="0 0 0" rpy="0 0 0"/>
           <geometry>
@@ -64,5 +64,5 @@
         </inertial>
         <visual>
-          <!-- FIXED: Remove large offset from visual origin -->
+          <!-- FIXED: Simplified visual origin - let joint handle positioning -->
           <origin xyz="0 0 0" rpy="0 0 0"/>
           <geometry>
@@ -72,5 +72,5 @@
         </visual>
         <collision name="left_finger_collision">
-          <!-- FIXED: Remove large offset from collision origin -->
+          <!-- FIXED: Simplified collision origin -->
           <origin xyz="0 0 0" rpy="0 0 0"/>
           <geometry>
@@ -79,7 +79,93 @@
         </collision>
       </link>
-      <!-- FIXED: Joint origins positioned correctly relative to base -->
+      <!-- FIXED: Joint origins position fingers correctly relative to base -->
+      <!-- Left finger starts at closed position (35mm total opening) -->
       <joint name="left_finger_joint" type="prismatic">
-        <origin xyz="0.032 0.0 0.0" rpy="0 0 0"/>
+        <origin xyz="0.0175 0.0 0.0" rpy="0 0 0"/>
+        <parent link="${prefix}base_link"/>
+        <child link="${prefix}left_finger_link"/>
+        <axis xyz="-1.0 0.0 0.0"/>
+        <!-- 0mm to 20mm per finger (35mm to 75mm total opening) -->
+        <limit lower="0.0" upper="0.020" effort="140" velocity="0.45"/>
+      </joint>
+      <!-- Right finger starts at closed position (mirrors left finger) -->
+      <joint name="right_finger_joint" type="prismatic">
+        <origin xyz="-0.0175 0.0 0.0" rpy="0 0 0"/>
+        <parent link="${prefix}base_link"/>
+        <child link="${prefix}right_finger_link"/>
+        <axis xyz="1.0 0.0 0.0"/>
+        <!-- -20mm to 0mm per finger (mirror of left finger) -->
+        <limit lower="-0.020" upper="0.0" effort="140" velocity="0.45"/>
+        <mimic joint="left_finger_joint" multiplier="1.0"/>
+      </joint>
+    </xacro:if>
+    <xacro:if value="${config == 'inwards'}">
+      <link name="${prefix}base_link">
+        <inertial>
+          <origin xyz="-4.8989159583623376e-05 2.847569602502098e-06 0.06811082379775064" rpy="0 0 0"/>
+          <mass value="1.2646523179240972"/>
+          <inertia ixx="0.001504" iyy="0.001812" izz="0.001053" ixy="-0.0" iyz="0.0" ixz="-3e-06"/>
+        </inertial>
+        <visual>
+          <origin xyz="0 0 0" rpy="0 0 0"/>
+          <geometry>
+            <mesh filename="package://onrobot_2fg7_gripper_description/meshes/base_link.stl" scale="0.001 0.001 0.001"/>
+          </geometry>
+          <material name="silver"/>
+        </visual>
+        <collision>
+          <origin xyz="0 0 0" rpy="0 0 0"/>
+          <geometry>
+            <mesh filename="package://onrobot_2fg7_gripper_description/meshes/base_link.stl" scale="0.001 0.001 0.001"/>
+          </geometry>
+        </collision>
+      </link>
+      <link name="${prefix}right_finger_link">
+        <inertial>
+          <origin xyz="0.029847703322119633 0.029496959480087837 0.015234215486232036" rpy="0 0 0"/>
+          <mass value="0.023219383355922288"/>
+          <inertia ixx="6e-06" iyy="5e-06" izz="2e-06" ixy="-0.0" iyz="0.0" ixz="-1e-06"/>
+        </inertial>
+        <visual>
+          <!-- FIXED: Simplified visual origin -->
+          <origin xyz="0 0 0" rpy="0 0 0"/>
+          <geometry>
+            <mesh filename="package://onrobot_2fg7_gripper_description/meshes/inwards/right_finger_link.stl" scale="0.001 0.001 0.001"/>
+          </geometry>
+          <material name="silver"/>
+        </visual>
+        <collision>
+          <!-- FIXED: Simplified collision origin -->
+          <origin xyz="0 0 0" rpy="0 0 0"/>
+          <geometry>
+            <mesh filename="package://onrobot_2fg7_gripper_description/meshes/inwards/right_finger_link.stl" scale="0.001 0.001 0.001"/>
+          </geometry>
+        </collision>
+      </link>
+      <link name="${prefix}left_finger_link">
+        <inertial>
+          <origin xyz="-0.007725703322151688 0.029491040519911117 0.015234215486238503" rpy="0 0 0"/>
+          <mass value="0.023219383355922288"/>
+          <inertia ixx="6e-06" iyy="5e-06" izz="2e-06" ixy="-0.0" iyz="-0.0" ixz="1e-06"/>
+        </inertial>
+        <visual>
+          <!-- FIXED: Simplified visual origin -->
+          <origin xyz="0 0 0" rpy="0 0 0"/>
+          <geometry>
+            <mesh filename="package://onrobot_2fg7_gripper_description/meshes/inwards/left_finger_link.stl" scale="0.001 0.001 0.001"/>
+          </geometry>
+          <material name="silver"/>
+        </visual>
+        <collision>
+          <!-- FIXED: Simplified collision origin -->
+          <origin xyz="0 0 0" rpy="0 0 0"/>
+          <geometry>
+            <mesh filename="package://onrobot_2fg7_gripper_description/meshes/inwards/left_finger_link.stl" scale="0.001 0.001 0.001"/>
+          </geometry>
+        </collision>
+      </link>
+      <!-- FIXED: Joint origins for inward configuration -->
+      <joint name="left_finger_joint" type="prismatic">
+        <origin xyz="0.0175 0.0 0.0" rpy="0 0 0"/>
         <parent link="${prefix}base_link"/>
         <child link="${prefix}left_finger_link"/>
@@ -88,5 +174,5 @@
       </joint>
       <joint name="right_finger_joint" type="prismatic">
-        <origin xyz="-0.032 0.0 0.0" rpy="0 0 0"/>
+        <origin xyz="-0.0175 0.0 0.0" rpy="0 0 0"/>
         <parent link="${prefix}base_link"/>
         <child link="${prefix}right_finger_link"/>

Commit message: xacro finger grips spawned fix

File: urdf/onrobot_2fg7.xacro (robot description, xacro)
@@ -158,6 +158,6 @@
         <child link="${prefix}left_finger_link"/>
         <axis xyz="-1.0 0.0 0.0"/>
-        <!-- CORRECTED: 0mm to 20mm per finger (35mm to 75mm total opening) -->
-        <limit lower="0.0" upper="0.020" effort="140" velocity="0.45"/>
+        <!-- CORRECTED: 0mm to 17.5mm per finger (35mm to 70mm total opening) -->
+        <limit lower="0.0" upper="0.0175" effort="140" velocity="0.45"/>
       </joint>
       <joint name="right_finger_joint" type="prismatic">
@@ -166,6 +166,6 @@
         <child link="${prefix}right_finger_link"/>
         <axis xyz="1.0 0.0 0.0"/>
-        <!-- CORRECTED: -20mm to 0mm per finger (mirror of left finger) -->
-        <limit lower="-0.020" upper="0.0" effort="140" velocity="0.45"/>
+        <!-- CORRECTED: -17.5mm to 0mm per finger (mirror of left finger) -->
+        <limit lower="-0.0175" upper="0.0" effort="140" velocity="0.45"/>
         <mimic joint="left_finger_joint" multiplier="1.0"/>
       </joint>

Commit message: xacro finger grips spawned fix

File: urdf/onrobot_2fg7.xacro (robot description, xacro)
@@ -42,5 +42,6 @@
         </inertial>
         <visual>
-          <origin xyz="0.054361 0.029494 -0.12005" rpy="0 0 0"/>
+          <!-- FIX: Rotated 180° around Z-axis and adjusted origin -->
+          <origin xyz="0.054361 0.029494 -0.12005" rpy="0 0 3.14159"/>
           <geometry>
             <mesh filename="package://onrobot_2fg7_gripper_description/meshes/right_finger_link.stl" scale="0.001 0.001 0.001"/>
@@ -49,5 +50,6 @@
         </visual>
         <collision name="right_finger_collision">
-          <origin xyz="0.054361 0.029494 -0.12005" rpy="0 0 0"/>
+          <!-- FIX: Same rotation as visual -->
+          <origin xyz="0.054361 0.029494 -0.12005" rpy="0 0 3.14159"/>
           <geometry>
             <mesh filename="package://onrobot_2fg7_gripper_description/meshes/right_finger_link.stl" scale="0.001 0.001 0.001"/>
@@ -62,5 +64,6 @@
         </inertial>
         <visual>
-          <origin xyz="-0.032239 0.029494 -0.12005" rpy="0 0 0"/>
+          <!-- FIX: Rotated 180° around Z-axis and adjusted origin -->
+          <origin xyz="-0.032239 0.029494 -0.12005" rpy="0 0 3.14159"/>
           <geometry>
             <mesh filename="package://onrobot_2fg7_gripper_description/meshes/left_finger_link.stl" scale="0.001 0.001 0.001"/>
@@ -69,5 +72,6 @@
         </visual>
         <collision name="left_finger_collision">
-          <origin xyz="-0.032239 0.029494 -0.12005" rpy="0 0 0"/>
+          <!-- FIX: Same rotation as visual -->
+          <origin xyz="-0.032239 0.029494 -0.12005" rpy="0 0 3.14159"/>
           <geometry>
             <mesh filename="package://onrobot_2fg7_gripper_description/meshes/left_finger_link.stl" scale="0.001 0.001 0.001"/>
@@ -75,16 +79,17 @@
         </collision>
       </link>
+      <!-- FIX: Joint origins and axes for proper alignment -->
       <joint name="left_finger_joint" type="prismatic">
-        <origin xyz="0.032239 -0.029494 0.12005" rpy="0 0 0"/>
+        <origin xyz="-0.032239 0.029494 0.12005" rpy="0 0 0"/>
         <parent link="${prefix}base_link"/>
         <child link="${prefix}left_finger_link"/>
-        <axis xyz="-1.0 0.0 0.0"/>
-        <limit lower="0.0" upper="0.019" effort="140" velocity="0.45"/> <!-- total 0.38 -->
+        <axis xyz="1.0 0.0 0.0"/>
+        <limit lower="0.0" upper="0.019" effort="140" velocity="0.45"/>
       </joint>
       <joint name="right_finger_joint" type="prismatic">
-        <origin xyz="-0.054361 -0.029494 0.12005" rpy="0 0 0"/>
+        <origin xyz="0.054361 0.029494 0.12005" rpy="0 0 0"/>
         <parent link="${prefix}base_link"/>
         <child link="${prefix}right_finger_link"/>
-        <axis xyz="1.0 0.0 0.0"/>
+        <axis xyz="-1.0 0.0 0.0"/>
         <limit lower="-0.019" upper="0.019" effort="140" velocity="0.45"/>
         <mimic joint="left_finger_joint" multiplier="1.0"/>
@@ -119,5 +124,6 @@
         </inertial>
         <visual>
-          <origin xyz="0.054361 0.029494 -0.12005" rpy="0 0 0"/>
+          <!-- FIX: Rotated 180° around Z-axis -->
+          <origin xyz="0.054361 0.029494 -0.12005" rpy="0 0 3.14159"/>
           <geometry>
             <mesh filename="package://onrobot_2fg7_gripper_description/meshes/inwards/right_finger_link.stl" scale="0.001 0.001 0.001"/>
@@ -126,5 +132,6 @@
         </visual>
         <collision>
-          <origin xyz="0.054361 0.029494 -0.12005" rpy="0 0 0"/>
+          <!-- FIX: Same rotation as visual -->
+          <origin xyz="0.054361 0.029494 -0.12005" rpy="0 0 3.14159"/>
           <geometry>
             <mesh filename="package://onrobot_2fg7_gripper_description/meshes/inwards/right_finger_link.stl" scale="0.001 0.001 0.001"/>
@@ -139,5 +146,6 @@
         </inertial>
         <visual>
-          <origin xyz="-0.032239 0.029494 -0.12005" rpy="0 0 0"/>
+          <!-- FIX: Rotated 180° around Z-axis -->
+          <origin xyz="-0.032239 0.029494 -0.12005" rpy="0 0 3.14159"/>
           <geometry>
             <mesh filename="package://onrobot_2fg7_gripper_description/meshes/inwards/left_finger_link.stl" scale="0.001 0.001 0.001"/>
@@ -146,5 +154,6 @@
         </visual>
         <collision>
-          <origin xyz="-0.032239 0.029494 -0.12005" rpy="0 0 0"/>
+          <!-- FIX: Same rotation as visual -->
+          <origin xyz="-0.032239 0.029494 -0.12005" rpy="0 0 3.14159"/>
           <geometry>
             <mesh filename="package://onrobot_2fg7_gripper_description/meshes/inwards/left_finger_link.stl" scale="0.001 0.001 0.001"/>
@@ -152,19 +161,17 @@
         </collision>
       </link>
-      <!-- For outward configuration -->
+      <!-- FIX: Joint origins and axes for proper alignment -->
       <joint name="left_finger_joint" type="prismatic">
-        <origin xyz="0.032239 -0.029494 0.12005" rpy="0 0 0"/>
+        <origin xyz="-0.032239 0.029494 0.12005" rpy="0 0 0"/>
         <parent link="${prefix}base_link"/>
         <child link="${prefix}left_finger_link"/>
-        <axis xyz="-1.0 0.0 0.0"/>
-        <!-- CORRECTED: 0mm to 17.5mm per finger (35mm to 70mm total opening) -->
+        <axis xyz="1.0 0.0 0.0"/>
         <limit lower="0.0" upper="0.0175" effort="140" velocity="0.45"/>
       </joint>
       <joint name="right_finger_joint" type="prismatic">
-        <origin xyz="-0.054361 -0.029494 0.12005" rpy="0 0 0"/>
+        <origin xyz="0.054361 0.029494 0.12005" rpy="0 0 0"/>
         <parent link="${prefix}base_link"/>
         <child link="${prefix}right_finger_link"/>
-        <axis xyz="1.0 0.0 0.0"/>
-        <!-- CORRECTED: -17.5mm to 0mm per finger (mirror of left finger) -->
+        <axis xyz="-1.0 0.0 0.0"/>
         <limit lower="-0.0175" upper="0.0" effort="140" velocity="0.45"/>
         <mimic joint="left_finger_joint" multiplier="1.0"/>

Commit message: Driver connectivity - fix package 1

File: urdf/onrobot_2fg7.xacro (robot description, xacro)
@@ -75,4 +75,5 @@
         </collision>
       </link>
+      <!-- FIXED: Consistent joint limits - 17.5mm per finger (35mm total opening) -->
       <joint name="left_finger_joint" type="prismatic">
         <origin xyz="0.032239 -0.029494 0.12005" rpy="0 0 0"/>
@@ -80,5 +81,6 @@
         <child link="${prefix}left_finger_link"/>
         <axis xyz="-1.0 0.0 0.0"/>
-        <limit lower="0.0" upper="0.019" effort="140" velocity="0.45"/> <!-- total 0.38 -->
+        <!-- CORRECTED: 0.0 to 0.0175m (17.5mm per finger, 35mm total opening) -->
+        <limit lower="0.0" upper="0.0175" effort="140" velocity="0.45"/>
       </joint>
       <joint name="right_finger_joint" type="prismatic">
@@ -87,5 +89,6 @@
         <child link="${prefix}right_finger_link"/>
         <axis xyz="1.0 0.0 0.0"/>
-        <limit lower="-0.019" upper="0.019" effort="140" velocity="0.45"/>
+        <!-- CORRECTED: -0.0175 to 0.0m (mirrored left finger) -->
+        <limit lower="-0.0175" upper="0.0" effort="140" velocity="0.45"/>
         <mimic joint="left_finger_joint" multiplier="1.0"/>
       </joint>
@@ -152,5 +155,5 @@
         </collision>
       </link>
-      <!-- For outward configuration -->
+      <!-- FIXED: Consistent joint limits for inward configuration -->
       <joint name="left_finger_joint" type="prismatic">
         <origin xyz="0.032239 -0.029494 0.12005" rpy="0 0 0"/>
@@ -158,5 +161,5 @@
         <child link="${prefix}left_finger_link"/>
         <axis xyz="-1.0 0.0 0.0"/>
-        <!-- CORRECTED: 0mm to 17.5mm per finger (35mm to 70mm total opening) -->
+        <!-- CORRECTED: 0.0 to 0.0175m (17.5mm per finger, 35mm total opening) -->
         <limit lower="0.0" upper="0.0175" effort="140" velocity="0.45"/>
       </joint>
@@ -166,5 +169,5 @@
         <child link="${prefix}right_finger_link"/>
         <axis xyz="1.0 0.0 0.0"/>
-        <!-- CORRECTED: -17.5mm to 0mm per finger (mirror of left finger) -->
+        <!-- CORRECTED: -0.0175 to 0.0m (mirrored left finger) -->
         <limit lower="-0.0175" upper="0.0" effort="140" velocity="0.45"/>
         <mimic joint="left_finger_joint" multiplier="1.0"/>
